File: Small_car_electronics&models/Small_car_electronics.FCStd/Small_car_electronics.FCStd.kicad_sch (KiCad schematic)
At the start: 12 parts, among them M1 Motor_Servo, M2 Motor_DC, M3 Motor_DC, SW1 SW_Wuerth_450301014042

Commit message: Updated design
Created better design for car shell and
car PCB, removed compass and changed plastic tracks to rubber belt.
Parts:
- removed GY-273_Compass1: ~, symbol Small_car_library:GY-273_Compass
Connections:
- net at TP4056_Module. (OUT-): now also SW1.1 (B)
- net at TB6612FNG_Motor_Driver. (GND): now also M3.2 (-)
- new net: MT3608_Step_Up_5V_Module. (VOUT-), TB6612FNG_Motor_Driver. (GND), TP4056_Module. (OUT-)
